File: schema esp201.sch (EAGLE design)
At the start: 9 parts

Commit message: +
Parts:
- added SL1: (no value), con-amp-quick:M02
- SL2: device con-amp-quick:M02 -> con-amp-quick:M04
Connections:
- net +12V: now also SL2.2
- net +3V3: now also SL1.1
- net GND: now also SL1.2, SL2.4
- net N$7: now also SL2.3; no longer SL2.2
Changed lines of the file:
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@@
 <?xml version="1.0" encoding="utf-8"?>
 <!DOCTYPE eagle SYSTEM "eagle.dtd">
-<eagle version="7.3.0">
+<eagle version="6.5.0">
 <drawing>
 <settings>
@@
 <part name="S1" library="switch-misc" deviceset="PVA1R" device=""/>
 <part name="P+1" library="supply1" deviceset="+12V" device=""/>
-<part name="SL2" library="con-amp-quick" deviceset="M02" device=""/>
 <part name="SL3" library="con-amp-quick" deviceset="M04" device=""/>
+<part name="SL1" library="con-amp-quick" deviceset="M02" device=""/>
+<part name="SL2" library="con-amp-quick" deviceset="M04" device=""/>
 </parts>
 <sheets>
@@
 <instance part="S1" gate="2" x="10.16" y="40.64"/>
 <instance part="P+1" gate="1" x="83.82" y="81.28"/>
-<instance part="SL2" gate="G$1" x="91.44" y="71.12" rot="R180"/>
 <instance part="SL3" gate="G$1" x="-10.16" y="71.12"/>
+<instance part="SL1" gate="G$1" x="76.2" y="71.12" rot="R180"/>
+<instance part="SL2" gate="G$1" x="101.6" y="71.12" rot="R180"/>
 </instances>
 <busses>
@@
 <wire x1="10.16" y1="35.56" x2="10.16" y2="33.02" width="0.1524" layer="91"/>
 <wire x1="10.16" y1="33.02" x2="20.32" y2="33.02" width="0.1524" layer="91"/>
+<pinref part="SL1" gate="G$1" pin="2"/>
+<wire x1="68.58" y1="68.58" x2="68.58" y2="50.8" width="0.1524" layer="91"/>
+<wire x1="83.82" y1="33.02" x2="96.52" y2="33.02" width="0.1524" layer="91"/>
+<wire x1="96.52" y1="33.02" x2="96.52" y2="66.04" width="0.1524" layer="91"/>
+<pinref part="SL2" gate="G$1" pin="4"/>
 </segment>
 </net>
@@
 <wire x1="20.32" y1="48.26" x2="20.32" y2="60.96" width="0.1524" layer="91"/>
 <wire x1="20.32" y1="60.96" x2="20.32" y2="81.28" width="0.1524" layer="91"/>
-<wire x1="20.32" y1="81.28" x2="73.66" y2="81.28" width="0.1524" layer="91"/>
+<wire x1="20.32" y1="81.28" x2="68.58" y2="81.28" width="0.1524" layer="91"/>
+<wire x1="68.58" y1="81.28" x2="73.66" y2="81.28" width="0.1524" layer="91"/>
 <wire x1="73.66" y1="81.28" x2="73.66" y2="86.36" width="0.1524" layer="91"/>
 <pinref part="U$1" gate="G$1" pin="CH_PD"/>
@@
 <pinref part="R4" gate="G$1" pin="1"/>
 <wire x1="10.16" y1="60.96" x2="20.32" y2="60.96" width="0.1524" layer="91"/>
+<pinref part="SL1" gate="G$1" pin="1"/>
+<wire x1="68.58" y1="71.12" x2="68.58" y2="81.28" width="0.1524" layer="91"/>
 </segment>
 </net>
@@
 </segment>
 </net>
+<net name="+12V" class="0">
+<segment>
+<pinref part="P+1" gate="1" pin="+12V"/>
+<wire x1="83.82" y1="78.74" x2="83.82" y2="73.66" width="0.1524" layer="91"/>
+<wire x1="83.82" y1="73.66" x2="96.52" y2="73.66" width="0.1524" layer="91"/>
+<pinref part="SL2" gate="G$1" pin="1"/>
+<pinref part="SL2" gate="G$1" pin="2"/>
+<wire x1="96.52" y1="73.66" x2="96.52" y2="71.12" width="0.1524" layer="91"/>
+</segment>
+</net>
 <net name="N$7" class="0">
 <segment>
 <pinref part="R1" gate="G$1" pin="1"/>
-<pinref part="SL2" gate="G$1" pin="2"/>
-</segment>
-</net>
-<net name="+12V" class="0">
-<segment>
-<pinref part="P+1" gate="1" pin="+12V"/>
-<pinref part="SL2" gate="G$1" pin="1"/>
-<wire x1="83.82" y1="78.74" x2="83.82" y2="71.12" width="0.1524" layer="91"/>
-</segment>
-</net>
+<pinref part="SL2" gate="G$1" pin="3"/>
+<wire x1="83.82" y1="68.58" x2="96.52" y2="68.58" width="0.1524" layer="91"/>
+</segment>
+</net>
