File: schema esp01.brd (EAGLE design)
At the start: 44.1 x 35.5 mm, 8 parts

Commit message: +
Parts:
- R1: value (none) -> 220
- R2: value (none) -> 10k
- R3: value (none) -> 2.2k
Changed lines of the file:
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@@
 <attribute name="MPN" value="" x="30.48" y="10.16" size="1.778" layer="27" rot="R270" display="off"/>
 </element>
-<element name="R1" library="rcl" package="0204/7" value="" x="19.05" y="15.24" rot="R270"/>
+<element name="R1" library="rcl" package="0204/7" value="220" x="19.05" y="15.24" rot="R270"/>
 <element name="X4" library="con-wago-508" package="W237-132" value="" x="3.81" y="27.94" rot="R90">
 <attribute name="MF" value="" x="3.81" y="27.94" size="1.778" layer="27" rot="R90" display="off"/>
@@
 <attribute name="MPN" value="" x="3.81" y="27.94" size="1.778" layer="27" rot="R90" display="off"/>
 </element>
-<element name="R2" library="rcl" package="0204/7" value="" x="11.43" y="16.51" rot="R90"/>
-<element name="R3" library="rcl" package="0204/7" value="" x="11.43" y="26.67" rot="R90"/>
+<element name="R2" library="rcl" package="0204/7" value="10k" x="11.43" y="16.51" rot="R90"/>
+<element name="R3" library="rcl" package="0204/7" value="2.2k" x="11.43" y="26.67" rot="R90"/>
 <element name="X5" library="con-wago-508" package="W237-4P" value="" x="5.08" y="12.7" rot="R270">
 <attribute name="MF" value="" x="5.08" y="12.7" size="1.778" layer="27" rot="R270" display="off"/>
