File: schema esp01-doma.brd (EAGLE design)
At the start: 44.1 x 35.5 mm, 8 parts

Commit message: +
Parts:
- R2: value 10k -> 20k
- R3: value 2.2k -> 6k8
Changed lines of the file:
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@@
 <attribute name="MPN" value="" x="3.81" y="27.94" size="1.778" layer="27" rot="R90" display="off"/>
 </element>
-<element name="R2" library="rcl" package="0204/7" value="10k" x="11.43" y="16.51" rot="R90"/>
-<element name="R3" library="rcl" package="0204/7" value="2.2k" x="11.43" y="26.67" rot="R90"/>
+<element name="R2" library="rcl" package="0204/7" value="20k" x="11.43" y="16.51" rot="R90"/>
+<element name="R3" library="rcl" package="0204/7" value="6k8" x="11.43" y="26.67" rot="R90"/>
 <element name="X5" library="con-wago-508" package="W237-4P" value="" x="5.08" y="12.7" rot="R270">
 <attribute name="MF" value="" x="5.08" y="12.7" size="1.778" layer="27" rot="R270" display="off"/>
