File: schema esp01-chata.sch (EAGLE design)
At the start: 8 parts

Commit message: +
Parts:
- removed R2: 10k, rcl:R-EU_0204/7
- removed R3: 2.2k, rcl:R-EU_0204/7
- removed X2, X4: (no value), con-wago-508:W237-02P
- removed X5: (no value), con-wago-508:W237-04P
- added 12V, 3V3, ELMER, LED: (no value), con-wago-508:W237-02P
- added OK1: PC817, optocoupler:PC817
- added R4: 560, rcl:R-EU_0204/7
- added R5: 10k, rcl:R-EU_0204/7
- renumbered X3 to UART
Connections:
- removed net N$1: R2.1, X5-3.KL
- new net N$4: OK1.A, R4.2
- new net N$8: ELMER-1.KL, R4.1
- net +12V: now also 12V-1.KL, ELMER-2.KL; no longer X5-1.KL, X5-2.KL
- net +3V3: now also 3V3-1.KL, R5.2; no longer X4-1.KL
- net GND: now also 12V-2.KL, 3V3-2.KL, LED-2.KL, OK1.C, OK1.EMIT; no longer R3.2, X2-2.KL, X4-2.KL, X5-4.KL
- net N$2: now also LED-1.KL; no longer X2-1.KL
- net N$7: now also OK1.COL, R5.1; no longer R2.2, R3.1
Other:
- moved on the sheet: R1

Commit message: zmeny eagle
Changed lines of the file:
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@@
 <?xml version="1.0" encoding="utf-8"?>
 <!DOCTYPE eagle SYSTEM "eagle.dtd">
-<eagle version="7.3.0">
+<eagle version="6.5.0">
 <drawing>
 <settings>
@@
 <net name="+3V3" class="0">
 <segment>
+<pinref part="R5" gate="G$1" pin="2"/>
+<pinref part="+3V2" gate="G$1" pin="+3V3"/>
+</segment>
+<segment>
 <pinref part="3V3" gate="-1" pin="KL"/>
-<pinref part="+3V1" gate="G$1" pin="+3V3"/>
+<pinref part="U$1" gate="G$1" pin="VCC"/>
 <wire x1="-25.4" y1="101.6" x2="-20.32" y2="101.6" width="0.1524" layer="91"/>
-<wire x1="-20.32" y1="101.6" x2="-20.32" y2="106.68" width="0.1524" layer="91"/>
-<pinref part="U$1" gate="G$1" pin="VCC"/>
 <wire x1="-20.32" y1="101.6" x2="12.7" y2="101.6" width="0.1524" layer="91"/>
 <wire x1="12.7" y1="101.6" x2="12.7" y2="83.82" width="0.1524" layer="91"/>
+<pinref part="+3V1" gate="G$1" pin="+3V3"/>
+<wire x1="-20.32" y1="106.68" x2="-20.32" y2="101.6" width="0.1524" layer="91"/>
+<junction x="-20.32" y="101.6"/>
 <pinref part="U$1" gate="G$1" pin="CH_PD"/>
 <wire x1="12.7" y1="78.74" x2="12.7" y2="83.82" width="0.1524" layer="91"/>
-</segment>
-<segment>
-<pinref part="R5" gate="G$1" pin="2"/>
-<pinref part="+3V2" gate="G$1" pin="+3V3"/>
+<junction x="12.7" y="83.82"/>
 </segment>
 </net>
@@
 <net name="N$7" class="0">
 <segment>
-<pinref part="OK1" gate="A" pin="COL"/>
 <pinref part="R5" gate="G$1" pin="1"/>
-<wire x1="40.64" y1="121.92" x2="45.72" y2="121.92" width="0.1524" layer="91"/>
 <wire x1="10.16" y1="109.22" x2="45.72" y2="109.22" width="0.1524" layer="91"/>
 <wire x1="45.72" y1="109.22" x2="45.72" y2="121.92" width="0.1524" layer="91"/>
@@
 <wire x1="12.7" y1="73.66" x2="10.16" y2="73.66" width="0.1524" layer="91"/>
 <wire x1="10.16" y1="73.66" x2="10.16" y2="109.22" width="0.1524" layer="91"/>
+<pinref part="OK1" gate="A" pin="COL"/>
+<wire x1="40.64" y1="121.92" x2="45.72" y2="121.92" width="0.1524" layer="91"/>
+<junction x="45.72" y="121.92"/>
 </segment>
 </net>
@@
 <net name="GND" class="0">
 <segment>
-<pinref part="U$1" gate="G$1" pin="GND"/>
-<wire x1="7.62" y1="53.34" x2="45.72" y2="53.34" width="0.1524" layer="91"/>
-<wire x1="45.72" y1="53.34" x2="45.72" y2="68.58" width="0.1524" layer="91"/>
+<wire x1="7.62" y1="53.34" x2="50.8" y2="53.34" width="0.1524" layer="91"/>
 <wire x1="7.62" y1="96.52" x2="7.62" y2="73.66" width="0.1524" layer="91"/>
-<pinref part="UART" gate="-1" pin="KL"/>
 <wire x1="7.62" y1="73.66" x2="7.62" y2="53.34" width="0.1524" layer="91"/>
-<wire x1="45.72" y1="68.58" x2="91.44" y2="68.58" width="0.1524" layer="91"/>
 <pinref part="GND1" gate="1" pin="GND"/>
 <junction x="7.62" y="53.34"/>
-<wire x1="-25.4" y1="73.66" x2="7.62" y2="73.66" width="0.1524" layer="91"/>
-<pinref part="12V" gate="-2" pin="KL"/>
 <pinref part="3V3" gate="-2" pin="KL"/>
 <wire x1="7.62" y1="96.52" x2="-7.62" y2="96.52" width="0.1524" layer="91"/>
+<pinref part="12V" gate="-2" pin="KL"/>
+<wire x1="-7.62" y1="96.52" x2="-25.4" y2="96.52" width="0.1524" layer="91"/>
+<wire x1="-25.4" y1="73.66" x2="7.62" y2="73.66" width="0.1524" layer="91"/>
+<junction x="7.62" y="73.66"/>
+<pinref part="UART" gate="-1" pin="KL"/>
+<pinref part="U$1" gate="G$1" pin="GND"/>
+<wire x1="45.72" y1="68.58" x2="50.8" y2="68.58" width="0.1524" layer="91"/>
+<wire x1="50.8" y1="68.58" x2="91.44" y2="68.58" width="0.1524" layer="91"/>
+<wire x1="50.8" y1="53.34" x2="50.8" y2="68.58" width="0.1524" layer="91"/>
+<junction x="50.8" y="68.58"/>
 <pinref part="LED" gate="-2" pin="KL"/>
-<wire x1="-7.62" y1="96.52" x2="-25.4" y2="96.52" width="0.1524" layer="91"/>
 <wire x1="-7.62" y1="58.42" x2="-25.4" y2="58.42" width="0.1524" layer="91"/>
 <wire x1="-7.62" y1="58.42" x2="-7.62" y2="96.52" width="0.1524" layer="91"/>
+<junction x="-7.62" y="96.52"/>
 </segment>
 <segment>
@@
 <pinref part="OK1" gate="A" pin="EMIT"/>
 <wire x1="40.64" y1="116.84" x2="50.8" y2="116.84" width="0.1524" layer="91"/>
-<wire x1="38.1" y1="104.14" x2="50.8" y2="104.14" width="0.1524" layer="91"/>
 <wire x1="50.8" y1="104.14" x2="50.8" y2="116.84" width="0.1524" layer="91"/>
-</segment>
-</net>
+<wire x1="50.8" y1="104.14" x2="38.1" y2="104.14" width="0.1524" layer="91"/>
+<junction x="38.1" y="104.14"/>
+</segment>
+</net>
