File: oddelovac.brd (EAGLE design)
At the start: 100 x 80 mm, 5 parts

Commit message: zmena pcb
Other:
- board size 100 x 80 mm -> 35.2 x 17.8 mm
Changed lines of the file:
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@@
 <board>
 <plain>
-<wire x1="0" y1="0" x2="100" y2="0" width="0" layer="20"/>
-<wire x1="100" y1="0" x2="100" y2="80" width="0" layer="20"/>
-<wire x1="100" y1="80" x2="0" y2="80" width="0" layer="20"/>
-<wire x1="0" y1="80" x2="0" y2="0" width="0" layer="20"/>
+<wire x1="0" y1="0" x2="35.23" y2="0" width="0" layer="20"/>
+<wire x1="35.23" y1="0" x2="35.23" y2="17.77" width="0" layer="20"/>
+<wire x1="35.23" y1="17.77" x2="0" y2="17.77" width="0" layer="20"/>
+<wire x1="0" y1="17.77" x2="0" y2="0" width="0" layer="20"/>
 </plain>
 <attributes>

Commit message: +
Parts:
- renumbered INPUT1 to OUTPUT
Changed lines of the file:
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@@
 <attribute name="OC_FARNELL" value="unknown" x="-17.78" y="-13.97" size="1.778" layer="27" rot="R270" display="off"/>
 </element>
-<element name="INPUT1" library="con-wago-508" package="W237-3E" value="" x="29.21" y="7.62" rot="R90">
+<element name="OUTPUT" library="con-wago-508" package="W237-3E" value="" x="29.21" y="7.62" rot="R90">
 <attribute name="OC_NEWARK" value="unknown" x="29.21" y="7.62" size="1.778" layer="27" rot="R90" display="off"/>
 <attribute name="MPN" value="" x="29.21" y="7.62" size="1.778" layer="27" rot="R90" display="off"/>
@@
 <contactref element="OK1" pad="2"/>
 <contactref element="OK1" pad="3"/>
-<contactref element="INPUT1" pad="1"/>
+<contactref element="OUTPUT" pad="1"/>
 <wire x1="17.78" y1="11.43" x2="17.78" y2="3.81" width="1.016" layer="16"/>
 <wire x1="29.845" y1="2.54" x2="20.32" y2="2.54" width="1.016" layer="16"/>
@@
 <contactref element="OK1" pad="4"/>
 <contactref element="R2" pad="1"/>
-<contactref element="INPUT1" pad="2"/>
+<contactref element="OUTPUT" pad="2"/>
 <wire x1="21.59" y1="13.97" x2="21.59" y2="16.51" width="1.016" layer="16"/>
 <wire x1="21.59" y1="16.51" x2="15.24" y2="16.51" width="1.016" layer="16"/>
@@
 <signal name="+3V3">
 <contactref element="R2" pad="2"/>
-<contactref element="INPUT1" pad="3"/>
+<contactref element="OUTPUT" pad="3"/>
 <wire x1="21.59" y1="6.35" x2="25.4" y2="6.35" width="1.016" layer="16"/>
 <wire x1="25.4" y1="6.35" x2="25.4" y2="12.7" width="1.016" layer="16"/>

Commit message: +hodnoty resistoru
Parts:
- R1: value (none) -> 1k
- R2: value (none) -> 560
Changed lines of the file:
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@@
 <?xml version="1.0" encoding="utf-8"?>
 <!DOCTYPE eagle SYSTEM "eagle.dtd">
-<eagle version="6.5.0">
+<eagle version="7.3.0">
 <drawing>
 <settings>
@@
 <pass name="Default">
 <param name="RoutingGrid" value="50mil"/>
+<param name="AutoGrid" value="1"/>
+<param name="Efforts" value="0"/>
+<param name="TopRouterVariant" value="1"/>
 <param name="tpViaShape" value="round"/>
 <param name="PrefDir.1" value="|"/>
@@
 <attribute name="OC_FARNELL" value="9707727" x="34.29" y="0" size="1.778" layer="27" display="off"/>
 </element>
-<element name="R1" library="rcl" package="0207/7" value="" x="11.43" y="10.16" rot="R270"/>
-<element name="R2" library="rcl" package="0207/7" value="" x="21.59" y="10.16" rot="R270"/>
+<element name="R1" library="rcl" package="0207/7" value="1k" x="11.43" y="10.16" rot="R270"/>
+<element name="R2" library="rcl" package="0207/7" value="560" x="21.59" y="10.16" rot="R270"/>
 <element name="INPUT" library="con-wago-508" package="W237-3E" value="" x="5.08" y="7.62" rot="R270">
 <attribute name="OC_NEWARK" value="unknown" x="-17.78" y="-13.97" size="1.778" layer="27" rot="R270" display="off"/>
