File: oddelovac.sch (EAGLE design)
At the start: 5 parts

Commit message: +
Parts:
- renumbered INPUT1 to OUTPUT
Changed lines of the file:
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@@
 <part name="+3V1" library="supply1" deviceset="+3V3" device=""/>
 <part name="INPUT" library="con-wago-508" deviceset="W237-3E" device=""/>
-<part name="INPUT1" library="con-wago-508" deviceset="W237-3E" device=""/>
+<part name="OUTPUT" library="con-wago-508" deviceset="W237-3E" device=""/>
 </parts>
 <sheets>
@@
 <instance part="INPUT" gate="-2" x="53.34" y="60.96"/>
 <instance part="INPUT" gate="-3" x="53.34" y="58.42"/>
-<instance part="INPUT1" gate="-1" x="96.52" y="43.18" rot="R180"/>
-<instance part="INPUT1" gate="-2" x="96.52" y="48.26" rot="R180"/>
-<instance part="INPUT1" gate="-3" x="96.52" y="53.34" rot="R180"/>
+<instance part="OUTPUT" gate="-1" x="96.52" y="43.18" rot="R180"/>
+<instance part="OUTPUT" gate="-2" x="96.52" y="48.26" rot="R180"/>
+<instance part="OUTPUT" gate="-3" x="96.52" y="53.34" rot="R180"/>
 </instances>
 <busses>
@@
 <wire x1="91.44" y1="43.18" x2="81.28" y2="43.18" width="0.1524" layer="91"/>
 <junction x="81.28" y="43.18"/>
-<pinref part="INPUT1" gate="-1" pin="KL"/>
+<pinref part="OUTPUT" gate="-1" pin="KL"/>
 </segment>
 </net>
@@
 <wire x1="81.28" y1="48.26" x2="91.44" y2="48.26" width="0.1524" layer="91"/>
 <junction x="81.28" y="48.26"/>
-<pinref part="INPUT1" gate="-2" pin="KL"/>
+<pinref part="OUTPUT" gate="-2" pin="KL"/>
 </segment>
 </net>
@@
 <pinref part="+3V1" gate="G$1" pin="+3V3"/>
 <wire x1="81.28" y1="60.96" x2="81.28" y2="58.42" width="0.1524" layer="91"/>
-<pinref part="INPUT1" gate="-3" pin="KL"/>
+<pinref part="OUTPUT" gate="-3" pin="KL"/>
 <wire x1="91.44" y1="53.34" x2="86.36" y2="53.34" width="0.1524" layer="91"/>
 <wire x1="86.36" y1="53.34" x2="86.36" y2="58.42" width="0.1524" layer="91"/>

Commit message: +hodnoty resistoru
Parts:
- R1: value (none) -> 1k
- R2: value (none) -> 560
Changed lines of the file:
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@@
 <?xml version="1.0" encoding="utf-8"?>
 <!DOCTYPE eagle SYSTEM "eagle.dtd">
-<eagle version="6.5.0">
+<eagle version="7.3.0">
 <drawing>
 <settings>
@@
 <part name="OK1" library="optocoupler" deviceset="PC817" device=""/>
 <part name="GND1" library="supply1" deviceset="GND" device=""/>
-<part name="R1" library="rcl" deviceset="R-EU_" device="0207/7"/>
-<part name="R2" library="rcl" deviceset="R-EU_" device="0207/7"/>
+<part name="R1" library="rcl" deviceset="R-EU_" device="0207/7" value="1k"/>
+<part name="R2" library="rcl" deviceset="R-EU_" device="0207/7" value="560"/>
 <part name="+3V1" library="supply1" deviceset="+3V3" device=""/>
 <part name="INPUT" library="con-wago-508" deviceset="W237-3E" device=""/>
